File: design/CP2102USB2UART/CP2102USB2UART.kicad_pcb (KiCad board)
At the start: 2 copper layers, 20.5 x 15.1 mm, 13 parts, among them J1 Conn_01x06, J2 UJ2-MIBH-G-SMT-TR, U1 CP2102

Commit message: bg top and bottom ready
Connections:
- R4 pad 1: unconnected-(R4-Pad1) -> VCC
Routing:
- net GND: track 30.1 -> 4.14 mm, vias 4 -> 0
- net VCC: track 22.9 -> 26.6 mm
- net Net-(U1-VBUS): track 4.95 -> 3.60 mm, vias 1 -> 0
- removed copper zone on B.Cu, net GND

Commit message: end of retroengineering
Parts:
- turned D1 to 90 degrees
Connections:
- net Net-(U1-~{SUSPEND}) renamed ~{SUSPEND}
- C2 pad 1: VCC -> VDD
- C3 pad 1: Net-(U1-VBUS) -> VCC
- D1 pad 1: Net-(D1-K) -> TXO
- D1 pad 2: TXD -> Net-(D1-A)
- J1 pad 1: 3v3 -> VDD
- J1 pad 4: TX0 -> TXO
- J1 pad 6: VCC -> +5V
- J2 pad 2: GND -> D-
- R1 pad 1: Net-(D1-K) -> VDD
- R1 pad 2: GND -> Net-(D1-A)
- R2 pad 1: 3v3 -> Net-(D2-A)
- R2 pad 2: Net-(D2-A) -> VDD
- R4 pad 1: VCC -> +5V
- R4 pad 2: GND -> VCC
- U1 pad 10: Net-(U1-NC-Pad10) -> unconnected-(U1-NC-Pad10)_7
- U1 pad 13: Net-(U1-NC-Pad10) -> unconnected-(U1-NC-Pad10)_1
- U1 pad 14: Net-(U1-NC-Pad10) -> unconnected-(U1-NC-Pad10)_9
- U1 pad 15: Net-(U1-NC-Pad10) -> unconnected-(U1-NC-Pad10)_4
- U1 pad 16: Net-(U1-NC-Pad10) -> unconnected-(U1-NC-Pad10)_3
- U1 pad 17: Net-(U1-NC-Pad10) -> unconnected-(U1-NC-Pad10)_2
- U1 pad 18: Net-(U1-NC-Pad10) -> unconnected-(U1-NC-Pad10)_10
- U1 pad 19: Net-(U1-NC-Pad10) -> unconnected-(U1-NC-Pad10)_8
- U1 pad 20: Net-(U1-NC-Pad10) -> unconnected-(U1-NC-Pad10)_6
- U1 pad 21: Net-(U1-NC-Pad10) -> unconnected-(U1-NC-Pad10)
- U1 pad 22: Net-(U1-NC-Pad10) -> unconnected-(U1-NC-Pad10)_5
- U1 pad 26: TXD -> TXO
- U1 pad 28: unconnected-(U1-DTR-Pad28) -> DTR
- U1 pad 5: GND -> D-
- U1 pad 6: VCC -> VDD
- U1 pad 8: Net-(U1-VBUS) -> VCC
- U1 pad 9: Net-(U1-VBUS) -> VCC
Routing:
- net VDD: track 0.00 -> 36.8 mm, vias 0 -> 2
- net GND: track 4.14 -> 24.5 mm, vias 0 -> 1
- net TXO: track 0.00 -> 19.7 mm, vias 0 -> 1
- net +5V: track 0.00 -> 17.7 mm, vias 0 -> 1
- net DTR: track 0.00 -> 13.5 mm, vias 0 -> 1
- net D-: track 0.00 -> 5.30 mm, vias 0 -> 2
- net TXD: track 3.70 -> 0.00 mm
- net Net-(U1-VBUS): track 3.60 -> 0.00 mm
- net Net-(D1-K): track 2.15 -> 0.00 mm
- net Net-(D1-A): track 0.00 -> 2.15 mm
- net RXI: track 15.9 -> 16.6 mm
- net VCC: track 26.6 -> 25.9 mm, vias 1 -> 3
- added copper zone on B.Cu, net GND
